Commit message: fix(lab): resolve step() crash and URDF inertia warnings
Three fixes:
1. pybullet_env reset(): instantiate self._tasks BEFORE _load_scene() — the scene
   loader iterates over self._tasks to get positions; on episode 2+ this was using
   stale task objects from the previous episode causing corrupt URDF loading.

2. loadURDF: add useFixedBase=True and URDF_ENABLE_CACHED_GRAPHICS_SHAPES — scene
   props (pots, switches) are static decorations, not physics actors.

3. assets/plant_pot.urdf, light_switch.urdf: add explicit <inertial mass=0> blocks
   to visual-only child links (foliage, paddle). Without this PyBullet falls back to
   mass=1 which makes the green sphere and yellow paddle act as 1kg physics bodies,
   causing immediate collision instability on step 1.

File: assets/light_switch.urdf (robot description, URDF)
Before this commit: robot light_switch, 2 links, 1 joints
Links:
- link paddle: mass None -> 0

File: assets/plant_pot.urdf (robot description, URDF)
Before this commit: robot plant_pot, 2 links, 1 joints
Links:
- link foliage: mass None -> 0
