Commit message: fix(lab): reliable 5/5 task completion + camera controls + visual overhaul
- Fix floor crashes: SPEED_LIMIT 30%→20%, all task targets z=1.0
- Fix user_debug_gui crash on episode 2+ (resetSimulation wipes sliders)
- Fix SweepFloorTask obs: use current_target waypoint, not spec.target_position
- Fix progress bar: use _current_wp_idx for sweep, engage_steps_done for others
- Fix debug item ID stale refs after reset (User debug draw failed)
- Raise is_at_target tolerance 0.5→1.0, sweep waypoint tol 0.6→0.9
- Add incompatible checkpoint detection in load_actor()
- Add keyboard camera controls: WASD pan, QE zoom, ZX rotate, RF pitch, 0-5 presets
- Add follow-drone mode (0 key cycles through drones)
- Add drone visual overrides: 0.45m coloured discs, 8 distinct colours
- Add rich HUD: task name, unicode progress bars, task-coloured labels
- Add floor tile (warm cream), ceiling (translucent), warm plaster walls
- Scale up URDF assets (plant_pot 3×, light_switch 5×, floor_zone 1.5×)
- Add obs_noise_std domain randomisation to HomeEnv (default off)
- Update README: correct deploy command, camera controls table

File: assets/floor_zone.urdf (robot description, URDF)
Before this commit: robot floor_zone, 1 links, 0 joints
Links:
- link zone: geometry visual box size=3.0 3.0 0.04

File: assets/light_switch.urdf (robot description, URDF)
Before this commit: robot light_switch, 2 links, 1 joints
Links:
- link paddle: geometry visual box size=0.20 0.10 0.35
- link plate: geometry collision box size=0.40 0.12 0.60; visual box size=0.40 0.12 0.60
Joints:
- joint paddle_joint: origin xyz=0 0.035 0.02 rpy=0 0 0 -> xyz=0 0.115 0.10 rpy=0 0 0

File: assets/plant_pot.urdf (robot description, URDF)
Before this commit: robot plant_pot, 2 links, 1 joints
Links:
- link foliage: geometry visual sphere radius=0.45
- link pot: geometry collision cylinder length=0.55 radius=0.35; visual cylinder length=0.55 radius=0.35
Joints:
- joint foliage_joint: origin xyz=0 0 0.38 rpy=0 0 0 -> xyz=0 0 0.90 rpy=0 0 0
